File: _autosave-final_schematic.sch (KiCad schematic (older format))
At the start: 47 parts, among them J1 Battery Babysitter, J2 BB_SYSOFF, J3 BOOT0, J4 OLED Qwiic, J5 Programmer, J8 GPS_COAX, SW1 SW_Push_SESS, SW2 SW_Push_RADIO, SW3 SW_Push_RST, U1 STM32L476VGTx, U2 MTK3339, U3 RFM95W-868S2, U4 BNO055, U5 LT1129-3.3_SO8

Commit message: pcb checkpoint
Parts:
- J5: footprint Connector_PinHeader_1.00mm:PinHeader_1x02_P1.00mm_Vertical -> Connector_PinHeader_1.00mm:PinHeader_1x04_P1.00mm_Vertical
- R10, R11, R9: footprint Resistor_SMD:R_0603_1608Metric_Pad1.05x0.95mm_HandSolder -> Resistor_SMD:R_0603_1608Metric_Pad0.98x0.95mm_HandSolder
- SW3: footprint Hardware_Repo:SW_1825910-6-4 -> footprint_lib:SW_1825910-6-4
Changed lines of the file:
@@
 EESchema Schematic File Version 4
-LIBS:final_schematic-cache
 EELAYER 30 0
 EELAYER END
@@
 F 0 "R10" H 1093 1150 50  0000 L BNN
 F 1 "62" H 1184 1150 50  0000 C TNN
-F 2 "Resistor_SMD:R_0603_1608Metric_Pad1.05x0.95mm_HandSolder" V 1230 1150 50  0001 C CNN
+F 2 "Resistor_SMD:R_0603_1608Metric_Pad0.98x0.95mm_HandSolder" V 1230 1150 50  0001 C CNN
 F 3 "~" H 1300 1150 50  0001 C CNN
 	1    1300 1150
@@
 $EndComp
 Text GLabel 9350 3600 0    50   Input ~ 0
-USART_RX
 Text GLabel 9350 3700 0    50   Input ~ 0
 USART_TX
@@
 F 0 "SW3" H 1050 4835 50  0000 C CNN
 F 1 "SW_Push_RST" H 1050 4744 50  0000 C CNN
-F 2 "Hardware_Repo:SW_1825910-6-4" H 1050 4750 50  0001 C CNN
+F 2 "footprint_lib:SW_1825910-6-4" H 1050 4750 50  0001 C CNN
 F 3 "" H 1050 4750 50  0001 C CNN
 	1    1050 4550
@@
 F 0 "R9" H 1093 3350 50  0000 L BNN
 F 1 "62" H 1184 3350 50  0000 C TNN
-F 2 "Resistor_SMD:R_0603_1608Metric_Pad1.05x0.95mm_HandSolder" V 1230 3350 50  0001 C CNN
+F 2 "Resistor_SMD:R_0603_1608Metric_Pad0.98x0.95mm_HandSolder" V 1230 3350 50  0001 C CNN
 F 3 "~" H 1300 3350 50  0001 C CNN
 	1    1300 3350
@@
 F 0 "R11" H 1243 4550 50  0000 L BNN
 F 1 "62" H 1334 4550 50  0000 C TNN
-F 2 "Resistor_SMD:R_0603_1608Metric_Pad1.05x0.95mm_HandSolder" V 1380 4550 50  0001 C CNN
+F 2 "Resistor_SMD:R_0603_1608Metric_Pad0.98x0.95mm_HandSolder" V 1380 4550 50  0001 C CNN
 F 3 "~" H 1450 4550 50  0001 C CNN
 	1    1450 4550
@@
 F 0 "J5" H 7868 1775 50  0000 C CNN
 F 1 "Programmer" H 7868 1866 50  0000 C CNN
-F 2 "Connector_PinHeader_1.00mm:PinHeader_1x02_P1.00mm_Vertical" H 7950 2200 50  0001 C CNN
+F 2 "Connector_PinHeader_1.00mm:PinHeader_1x04_P1.00mm_Vertical" H 7950 2200 50  0001 C CNN
 F 3 "~" H 7950 2200 50  0001 C CNN
 	1    7950 2200
