File: final_schematic_OLD.kicad_pcb (KiCad board)
At the start: 2 copper layers, 79.7 x 54.1 mm, 50 parts, among them J1 BB_COM_Conn_01x04_Male, J2 BB_CTRL_Conn_01x02_Male, J3 BB_ON/OFF_Conn_01x04_Male, J4 BOOT0_Conn_Male, J5 OLED_SPI_Conn_01x04_Male, J6 OLED_EN_Conn_01x02_Male, J7 Conn_ARM_JTAG_SWD_10, J8 GPS_COAX, SW1 SW_Push_SESS, SW2 SW_Push_RADIO, SW3 SW_Push_RST, U1 STM32L476VGTx, U2 MTK3339, U3 RFM95W-868S2, U4 BNO055

Commit message: I think this is going well
Parts:
- removed J6: OLED_EN_Conn_01x02_Male, Connector_PinHeader_1.00mm:PinHeader_1x01_P1.00mm_Vertical
- removed J7: Conn_ARM_JTAG_SWD_10, Connector_PinHeader_1.27mm:PinHeader_2x05_P1.27mm_Vertical_SMD
- removed R7, R8: 2.2k, Resistor_SMD:R_0603_1608Metric_Pad0.98x0.95mm_HandSolder
- removed RED1: LED_GPS_R, Diode_SMD:D_0603_1608Metric_Pad1.05x0.95mm_HandSolder
- added R11: 62, Resistor_SMD:R_0603_1608Metric_Pad0.98x0.95mm_HandSolder, F.Cu at (150.1, 106.7)
- added REF**: MountingHole_2.1mm, MountingHole:MountingHole_2.1mm, F.Cu at (143.2, 97.8)
- added REF**: MountingHole_2.1mm, MountingHole:MountingHole_2.1mm, F.Cu at (116.6, 97.8)
- added REF**: MountingHole_2.1mm, MountingHole:MountingHole_2.1mm, F.Cu at (143.2, 67.7)
- added REF**: MountingHole_2.1mm, MountingHole:MountingHole_2.1mm, F.Cu at (116.6, 67.7)
- added U5: LT1129-3.3_SO8, Package_SO:SOIC-8_3.9x4.9mm_P1.27mm, F.Cu at (128.0, 106.0)
- C10, C11, C14, C15, C16, C17, C2, C3, C4, C5, C6, C7, C8, C9: moved to B.Cu
- C12: value 1uF -> 3.3uF; footprint Capacitor_SMD:C_0603_1608Metric_Pad1.08x0.95mm_HandSolder -> Capacitor_Tantalum_SMD:CP_EIA-7343-15_Kemet-W_Pad2.25x2.55mm_HandSolder
- J1: value BB_COM_Conn_01x04_Male -> Battery Babysitter; footprint Connector_PinHeader_1.00mm:PinHeader_1x04_P1.00mm_Vertical -> Connector_PinHeader_1.00mm:PinHeader_1x06_P1.00mm_Vertical
- J2: value BB_CTRL_Conn_01x02_Male -> BB_SYSOFF
- J3: value BB_ON/OFF_Conn_01x04_Male -> BOOT0; footprint Connector_PinHeader_1.00mm:PinHeader_1x01_P1.00mm_Vertical -> Connector_PinHeader_1.00mm:PinHeader_1x02_P1.00mm_Vertical
- J4: value BOOT0_Conn_Male -> OLED Qwiic; footprint Connector_PinHeader_1.00mm:PinHeader_1x01_P1.00mm_Vertical -> Connector_JST:JST_EH_S4B-EH_1x04_P2.50mm_Horizontal
- J5: value OLED_SPI_Conn_01x04_Male -> Programmer; footprint Connector_PinHeader_1.00mm:PinHeader_1x06_P1.00mm_Vertical -> Connector_PinHeader_1.00mm:PinHeader_1x04_P1.00mm_Vertical
- R1, R2: value 48 -> 62
- R10: value 1k -> 62; footprint Resistor_SMD:R_0402_1005Metric_Pad0.72x0.64mm_HandSolder -> Resistor_SMD:R_0603_1608Metric_Pad0.98x0.95mm_HandSolder
- R9: value 10k -> 62
- SW3: footprint Button_Switch_SMD:SW_SPST_PTS645 -> footprint_lib:SW_1825910-6-4
- moved R9 109.9 mm to (168.4, 106.8)
- moved C2 92.0 mm to (166.8, 111.1), turned to 90 degrees
- moved C3 90.0 mm to (154.1, 109.0), turned to 180 degrees
- moved R5 88.6 mm to (154.1, 106.7)
- moved SW3 88.0 mm to (154.2, 111.2), turned to 0 degrees
- moved SW2 87.6 mm to (165.0, 111.2), turned to 0 degrees
- moved J2 86.5 mm to (136.0, 94.7), turned to 90 degrees
- moved R4 83.6 mm to (160.1, 106.9), turned to 0 degrees
- moved S1 76.9 mm to (131.2, 112.5)
- moved D1 75.6 mm to (120.2, 61.3), turned to 90 degrees
- moved C8 75.0 mm to (138.0, 88.9), turned to 270 degrees
- moved C6 74.3 mm to (137.5, 79.7), turned to 270 degrees
- moved J1 74.3 mm to (122.6, 108.8)
- moved C10 70.9 mm to (134.8, 90.1), turned to 180 degrees
- moved R1 70.0 mm to (120.2, 65.0), turned to 90 degrees
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Connections:
- C1 pad 2: PB1 -> Net-(C1-Pad2)
- C12 pad 1: Net-(C12-Pad1) -> 3V3
- C15 pad 1: 3V3 -> GND
- C15 pad 2: GND -> 3V3
- C2 pad 2: PB0 -> Net-(C2-Pad2)
- C3 pad 2: NRST -> Net-(C3-Pad2)
- J1 pad 3: I2C2_SDA -> I2C3_SDA
- J1 pad 4: I2C2_SCL -> I2C3_SCL
- J2 pad 1: PB12 -> GND
- J2 pad 2: PB13 -> SYSOFF
- J3 pad 1: PB14 -> BOOT0
- J4 pad 1: BOOT0 -> GND
- J5 pad 3: SPI1_MOSI -> SWDIO
- J5 pad 4: SPI1_SCK -> SWCLK
- R10 pad 1: Net-(R10-Pad1) -> session_btn
- R10 pad 2: GND -> Net-(C1-Pad2)
- R3 pad 2: PB1 -> Net-(C1-Pad2)
- R4 pad 2: PB0 -> Net-(C2-Pad2)
- R5 pad 2: NRST -> Net-(C3-Pad2)
- R9 pad 1: 3V3 -> radio_btn
- R9 pad 2: Net-(C12-Pad1) -> Net-(C2-Pad2)
- Re1 pad 2: PE0 -> IMU_nRST
- S1 pad 2: 3V3 -> BB_Out
- SW1 pad 1: PB1 -> Net-(C1-Pad2)
- SW2 pad 1: PB0 -> Net-(C2-Pad2)
- SW3 pad 1: NRST -> Net-(C3-Pad2)
- U1 pad 1: Net-(U1-Pad1) -> session_btn
- U1 pad 12: PH0 -> Net-(U1-Pad12)
- U1 pad 13: PH1 -> Net-(U1-Pad13)
- U1 pad 15: Net-(U1-Pad15) -> I2C3_SCL
- U1 pad 16: Net-(U1-Pad16) -> I2C3_SDA
- U1 pad 17: Net-(U1-Pad17) -> BB_CE
- U1 pad 18: Net-(U1-Pad18) -> BB_GPOUT
- U1 pad 2: PE3 -> radio_btn
- U1 pad 23: Net-(U1-Pad23) -> SYSOFF
- U1 pad 26: PA3 -> Net-(U1-Pad26)
- U1 pad 29: CS_OLED -> Net-(U1-Pad29)
- U1 pad 33: Net-(U1-Pad33) -> LoRa_RST
- U1 pad 34: Net-(U1-Pad34) -> CS_LORA
- U1 pad 35: PB0 -> Net-(U1-Pad35)
- U1 pad 36: PB1 -> Net-(U1-Pad36)
- U1 pad 43: CS_LORA -> IMU_ADDR
- U1 pad 44: Net-(U1-Pad44) -> BL_IND
- U1 pad 45: Net-(U1-Pad45) -> IMU_INT
- U1 pad 46: Net-(U1-Pad46) -> IMU_nRST
- U1 pad 51: PB12 -> Net-(U1-Pad51)
- U1 pad 52: PB13 -> Net-(U1-Pad52)
- U1 pad 53: PB14 -> Net-(U1-Pad53)
- U1 pad 67: DC_OLED -> Net-(U1-Pad67)
- U1 pad 68: Net-(U1-Pad68) -> USART_TX
- U1 pad 69: Net-(U1-Pad69) -> USART_RX
- U1 pad 85: USART_TX -> Net-(U1-Pad85)
- U1 pad 86: USART_RX -> Net-(U1-Pad86)
- U1 pad 89: SWO -> Net-(U1-Pad89)
- U1 pad 92: I2C_SCL -> I2C1_SCL
- U1 pad 93: I2C_SDA -> I2C1_SDA
- U1 pad 97: PE0 -> Net-(U1-Pad97)
- U2 pad 9: USART_RX -> N-00000104
- U3 pad 6: PA3 -> LoRa_RST
- U4 pad 10: PH1 -> BL_IND
- U4 pad 11: PE0 -> IMU_nRST
- U4 pad 14: PE3 -> IMU_INT
- U4 pad 17: PH0 -> IMU_ADDR
- U4 pad 19: I2C_SCL -> I2C2_SCL
- U4 pad 20: I2C_SDA -> I2C2_SDA
Routing:
- net GND: track 235.8 -> 16.5 mm
- net 3V3: track 159.1 -> 108.7 mm
- net I2C2_SDA: track 0.00 -> 39.0 mm
- net I2C2_SCL: track 0.00 -> 31.9 mm
- net NRST: track 16.9 -> 0.00 mm
- net PB0: track 16.7 -> 0.00 mm
- net I2C1_SCL: track 0.00 -> 15.8 mm
- net I2C1_SDA: track 0.00 -> 14.6 mm
- net IMU_ADDR: track 0.00 -> 13.5 mm
- net IMU_nRST: track 0.00 -> 12.1 mm
- net IMU_INT: track 0.00 -> 11.7 mm
- net Net-(C12-Pad1): track 9.77 -> 0.00 mm
- net PB1: track 8.37 -> 0.00 mm
- net Net-(J8-Pad1): track 7.82 -> 0.00 mm
- net I2C_SCL: track 7.77 -> 0.00 mm
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Other:
- board outline removed
