File: final_schematic.sch (KiCad schematic (older format))
At the start: 49 parts, among them J1 Battery Babysitter, J2 BB_SYSOFF, J3 BOOT0, J4 OLED Qwiic, J5 Programmer, J8 GPS_COAX, SW1 SW_Push_SESS, SW2 SW_Push_RADIO, SW3 SW_Push_RST, U1 STM32L476VGTx, U2 MTK3339, U3 RFM95W-868S2, U4 BNO055, U5 LT1129-3.3_SO8

Commit message: Schematic FINAL 	modified:   final_schematic-cache.lib 	modified:   final_schematic.sch 	modified:   final_schematic.sch-bak
Connections:
- net Text GLabel 9350 3700 0    50   Input ~ 0 is gone; now on net USART_RX: U2.9 (TX)
- net BB_CE: now also U1.13 (PH1); no longer U1.17 (PC2)
- net BB_GPOUT: now also U1.12 (PH0); no longer U1.18 (PC3)
- net BL_IND: now also U1.46 (PE15); no longer U1.44 (PE13)
- net CS_LORA: now also U1.29 (PA4); no longer U1.34 (PC5)
- net IMU_INT: now also U1.44 (PE13); no longer U1.45 (PE14)
- net IMU_nRST: now also U1.45 (PE14); no longer U1.46 (PE15)
- net LoRa_RST: now also U1.26 (PA3); no longer U1.33 (PC4)
- net USART_TX: now also U2.10 (RX)
- net radio_btn: now also U1.25 (PA2); no longer U1.2 (PE3)
- net session_btn: now also U1.24 (PA1); no longer U1.1 (PE2)
Other:
- moved on the sheet: D3, J1, J2
Changed lines of the file:
@@
 EESchema Schematic File Version 4
-LIBS:final_schematic-cache
-EELAYER 26 0
+EELAYER 30 0
 EELAYER END
 $Descr A4 11693 8268
@@
 $EndComp
 Text GLabel 9350 3600 0    50   Input ~ 0
-Text GLabel 9350 3700 0    50   Input ~ 0
-USART_TX
+USART_RX
 $Comp
 L final_schematic-rescue:MTK3339-GPS-rescue U2
@@
 L Connector_Generic:Conn_01x06 J1
 U 1 1 5FF26B1F
-P 800 6650
-F 0 "J1" H 906 6928 50  0000 C CNN
-F 1 "Battery Babysitter" V 906 6837 50  0000 R CNN
-F 2 "Connector_PinHeader_1.00mm:PinHeader_1x06_P1.00mm_Vertical" H 800 6650 50  0001 C CNN
-F 3 "~" H 800 6650 50  0001 C CNN
-	1    800  6650
+P 800 6550
+F 0 "J1" H 906 6828 50  0000 C CNN
+F 1 "Battery Babysitter" V 906 6737 50  0000 R CNN
+F 2 "Connector_PinHeader_1.00mm:PinHeader_1x06_P1.00mm_Vertical" H 800 6550 50  0001 C CNN
+F 3 "~" H 800 6550 50  0001 C CNN
+	1    800  6550
 	-1   0    0    1
 $EndComp
-Text Notes 850  6200 0    50   ~ 0
+Text Notes 850  6100 0    50   ~ 0
 Battery Babysitter \nConnector
+Text GLabel 1200 6550 2    50   Input ~ 0
+I2C3_SDA
+Text GLabel 1200 6450 2    50   Input ~ 0
+I2C3_SCL
 Text GLabel 1200 6650 2    50   Input ~ 0
-I2C3_SDA
-Text GLabel 1200 6550 2    50   Input ~ 0
-I2C3_SCL
-Text GLabel 1200 6750 2    50   Input ~ 0
 V_supply
 Wire Wire Line
-	1200 6750 1000 6750
-Wire Wire Line
 	1200 6650 1000 6650
+Wire Wire Line
+	1200 6550 1000 6550
 $Comp
 L power:GND #PWR05
 U 1 1 60007EB3
-P 1100 6850
-F 0 "#PWR05" H 1100 6600 50  0001 C CNN
-F 1 "GND" V 1105 6677 50  0000 C CNN
-F 2 "" H 1100 6850 50  0001 C CNN
-F 3 "" H 1100 6850 50  0001 C CNN
-	1    1100 6850
-	1    0    0    -1
-$EndComp
-Wire Wire Line
-	1200 6550 1000 6550
+P 1100 6750
+F 0 "#PWR05" H 1100 6500 50  0001 C CNN
+F 1 "GND" V 1105 6577 50  0000 C CNN
+F 2 "" H 1100 6750 50  0001 C CNN
+F 3 "" H 1100 6750 50  0001 C CNN
+	1    1100 6750
+	1    0    0    -1
+$EndComp
+Wire Wire Line
+	1200 6450 1000 6450
 Text Notes 8600 1700 2    50   ~ 10
 JTAG Debugger/Programmer
@@
 Text GLabel 9600 5500 0    50   Input ~ 0
 I2C2_SCL
-Text GLabel 1200 6450 2    50   Input ~ 0
+Text GLabel 1200 6350 2    50   Input ~ 0
 BB_GPOUT
 Wire Wire Line
-	1000 6350 1200 6350
-Wire Wire Line
-	1200 6450 1000 6450
+	1000 6250 1200 6250
+Wire Wire Line
+	1200 6350 1000 6350
 NoConn ~ 10600 3400
 NoConn ~ 10600 3500
@@
 Text GLabel 2800 1950 0    50   Input ~ 0
 3V3
-Text GLabel 3100 4650 0    50   Input ~ 0
+Text GLabel 3150 4850 0    50   Input ~ 0
 BL_IND
-Text GLabel 3100 4550 0    50   Input ~ 0
+Text GLabel 3150 4550 0    50   Input ~ 0
 IMU_ADDR
 Text GLabel 2600 1200 0    50   Input ~ 0
@@
 Text GLabel 5150 1650 2    50   Input ~ 0
 SYSOFF
-Text GLabel 5200 5350 2    50   Input ~ 0
+Text GLabel 3150 3050 0    50   Input ~ 0
 BB_GPOUT
-Text GLabel 3100 4850 0    50   Input ~ 0
+Text GLabel 3150 4750 0    50   Input ~ 0
 IMU_nRST
 NoConn ~ 3250 3450
@@
 NoConn ~ 5050 2850
 NoConn ~ 5050 2750
-NoConn ~ 5050 1850
-NoConn ~ 5050 1750
 NoConn ~ 4550 1350
 NoConn ~ 4450 1350
@@
 NoConn ~ 3250 3850
 NoConn ~ 3250 3750
-Text GLabel 3100 3550 0    50   Input ~ 0
+Text GLabel 5150 1750 2    50   Input ~ 0
 session_btn
-Text GLabel 3100 3650 0    50   Input ~ 0
+Text GLabel 5150 1850 2    50   Input ~ 0
 radio_btn
 Wire Wire Line
@@
 	4250 1250 4350 1250
 Connection ~ 4150 1250
-Text GLabel 3100 4750 0    50   Input ~ 0
+Text GLabel 3150 4650 0    50   Input ~ 0
 IMU_INT
-Text GLabel 5200 5550 2    50   Input ~ 0
+Text GLabel 5150 2050 2    50   Input ~ 0
 CS_LORA
-Text GLabel 5200 5450 2    50   Input ~ 0
+Text GLabel 5150 1950 2    50   Input ~ 0
 LoRa_RST
-Text GLabel 5200 5250 2    50   Input ~ 0
+Text GLabel 3150 3150 0    50   Input ~ 0
 BB_CE
-Text GLabel 5200 4450 2    50   Input ~ 0
+Text GLabel 5150 4450 2    50   Input ~ 0
 I2C2_SDA
-Text GLabel 5200 4350 2    50   Input ~ 0
+Text GLabel 5150 4350 2    50   Input ~ 0
 I2C2_SCL
 Connection ~ 4350 6950
@@
 Wire Wire Line
 	9050 5600 9600 5600
-Text GLabel 1200 6350 2    50   Input ~ 0
+Text GLabel 1200 6250 2    50   Input ~ 0
 BB_CE
 Wire Wire Line
@@
 L Connector_Generic:Conn_01x02 J2
 U 1 1 5FC7E508
-P 800 7550
-F 0 "J2" H 880 7542 50  0000 L CNN
-F 1 "BB_SYSOFF" V 880 7451 50  0000 R CNN
-F 2 "Connector_PinHeader_1.00mm:PinHeader_1x02_P1.00mm_Vertical" H 800 7550 50  0001 C CNN
-F 3 "~" H 800 7550 50  0001 C CNN
-	1    800  7550
+P 800 7500
+F 0 "J2" H 880 7492 50  0000 L CNN
+F 1 "BB_SYSOFF" V 880 7401 50  0000 R CNN
+F 2 "Connector_PinHeader_1.00mm:PinHeader_1x02_P1.00mm_Vertical" H 800 7500 50  0001 C CNN
+F 3 "~" H 800 7500 50  0001 C CNN
+	1    800  7500
 	-1   0    0    1
 $EndComp
@@
 L power:GND #PWR?
 U 1 1 5FC7E50E
-P 1000 7550
+P 1000 7500
 AR Path="/5F775B0B/5FC7E50E" Ref="#PWR?"  Part="1"
 AR Path="/5FC7E50E" Ref="#PWR0104"  Part="1"
-F 0 "#PWR0104" H 1000 7300 50  0001 C CNN
-F 1 "GND" H 1005 7377 50  0000 C CNN
-F 2 "" H 1000 7550 50  0001 C CNN
-F 3 "" H 1000 7550 50  0001 C CNN
-	1    1000 7550
-	1    0    0    -1
-$EndComp
-Text GLabel 1000 7450 2    50   Input ~ 0
+F 0 "#PWR0104" H 1000 7250 50  0001 C CNN
+F 1 "GND" H 1005 7327 50  0000 C CNN
+F 2 "" H 1000 7500 50  0001 C CNN
+F 3 "" H 1000 7500 50  0001 C CNN
+	1    1000 7500
+	1    0    0    -1
+$EndComp
+Text GLabel 1000 7400 2    50   Input ~ 0
 SYSOFF
 $Comp
@@
 NoConn ~ 6500 5750
 NoConn ~ 9350 3200
-NoConn ~ 5050 2050
 NoConn ~ 5050 2450
 NoConn ~ 5050 3650
 Wire Wire Line
-	1100 6850 1000 6850
+	1100 6750 1000 6750
 Wire Wire Line
 	7300 5750 7350 5750
@@
 	600  2450 600  2500
 Connection ~ 600  2450
-Text GLabel 5200 4050 2    50   Input ~ 0
+Text GLabel 5150 4050 2    50   Input ~ 0
 I2C1_SDA
-Text GLabel 5200 3950 2    50   Input ~ 0
+Text GLabel 5150 3950 2    50   Input ~ 0
 I2C1_SCL
-Text GLabel 5200 5150 2    50   Input ~ 0
+Text GLabel 5150 5150 2    50   Input ~ 0
 I2C3_SDA
-Text GLabel 5200 5050 2    50   Input ~ 0
+Text GLabel 5150 5050 2    50   Input ~ 0
 I2C3_SCL
 Wire Wire Line
@@
 Wire Wire Line
 	5050 3050 5150 3050
-Wire Wire Line
-	5200 3950 5050 3950
-Wire Wire Line
-	5050 4050 5200 4050
-Wire Wire Line
-	5200 4350 5050 4350
-Wire Wire Line
-	5050 4450 5200 4450
-Wire Wire Line
-	5200 5050 5050 5050
-Wire Wire Line
-	5050 5150 5200 5150
-Wire Wire Line
-	5200 5250 5050 5250
-Wire Wire Line
-	5200 5350 5050 5350
-Wire Wire Line
-	5200 5450 5050 5450
-Wire Wire Line
-	5200 5550 5050 5550
-Wire Wire Line
-	3100 3550 3250 3550
-Wire Wire Line
-	3250 3650 3100 3650
-Wire Wire Line
-	3100 4550 3250 4550
-Wire Wire Line
-	3250 4650 3100 4650
-Wire Wire Line
-	3100 4750 3250 4750
-Wire Wire Line
-	3250 4850 3100 4850
 Wire Wire Line
 	4350 1250 5800 1250
 Connection ~ 4350 1250
-NoConn ~ 5050 1950
 NoConn ~ 5050 3350
 NoConn ~ 5050 3450
-NoConn ~ 3250 3050
-NoConn ~ 3250 3150
 NoConn ~ 3250 3350
 NoConn ~ 5050 4550
@@
 L Device:D_Zener D3
 U 1 1 5F894344
-P 7800 4750
-F 0 "D3" H 7800 4966 50  0000 C CNN
-F 1 "D_Zener" H 7800 4875 50  0000 C CNN
-F 2 "footprint_lib:1N5355BRLG" H 7800 4750 50  0001 C CNN
-F 3 "~" H 7800 4750 50  0001 C CNN
-	1    7800 4750
-	1    0    0    -1
-$EndComp
-Text GLabel 8200 4750 2    50   Input ~ 0
+P 8300 4850
+F 0 "D3" H 8300 5066 50  0000 C CNN
+F 1 "D_Zener" H 8300 4975 50  0000 C CNN
+F 2 "footprint_lib:1N5355BRLG" H 8300 4850 50  0001 C CNN
+F 3 "~" H 8300 4850 50  0001 C CNN
+	1    8300 4850
+	1    0    0    -1
+$EndComp
+Text GLabel 8450 4850 2    50   Input ~ 0
 3V3
 $Comp
 L power:GND #PWR010
 U 1 1 5F8944C0
-P 7500 4750
-F 0 "#PWR010" H 7500 4500 50  0001 C CNN
-F 1 "GND" H 7505 4577 50  0000 C CNN
-F 2 "" H 7500 4750 50  0001 C CNN
-F 3 "" H 7500 4750 50  0001 C CNN
-	1    7500 4750
-	1    0    0    -1
-$EndComp
-Wire Wire Line
-	7650 4750 7500 4750
-Wire Wire Line
-	8200 4750 7950 4750
+P 8000 4850
+F 0 "#PWR010" H 8000 4600 50  0001 C CNN
+F 1 "GND" H 8005 4677 50  0000 C CNN
+F 2 "" H 8000 4850 50  0001 C CNN
+F 3 "" H 8000 4850 50  0001 C CNN
+	1    8000 4850
+	1    0    0    -1
+$EndComp
+Wire Wire Line
+	8150 4850 8000 4850
 $Comp
 L Device:CP1 C19
@@
 Wire Notes Line
 	6000 6400 11200 6400
-Wire Notes Line
-	7350 5100 7350 4250
-Wire Notes Line
-	7350 4250 11200 4250
-Text Notes 8050 4400 0    50   ~ 0
+Text Notes 8000 4550 0    50   ~ 0
 Surge protector
+Text GLabel 9350 3700 0    50   Input ~ 0
+USART_TX
+Wire Notes Line
+	11200 4250 8700 4250
+Wire Notes Line
+	8700 4400 7850 4400
+Wire Notes Line
+	7850 4400 7850 5100
+Wire Notes Line
+	1850 5850 450  5850
+Wire Wire Line
+	5050 1750 5150 1750
+Wire Wire Line
+	5050 1850 5150 1850
+Wire Wire Line
+	5050 1950 5150 1950
+Wire Wire Line
+	5050 2050 5150 2050
+Wire Wire Line
+	5150 3950 5050 3950
+Wire Wire Line
+	5050 4050 5150 4050
+Wire Wire Line
+	5150 4350 5050 4350
+Wire Wire Line
+	5050 4450 5150 4450
+Wire Wire Line
+	5150 5050 5050 5050
+Wire Wire Line
+	5050 5150 5150 5150
+Wire Wire Line
+	3250 4550 3150 4550
+Wire Wire Line
+	3150 4650 3250 4650
+Wire Wire Line
+	3250 4750 3150 4750
+Wire Wire Line
+	3150 4850 3250 4850
+Wire Wire Line
+	3250 3050 3150 3050
+Wire Wire Line
+	3150 3150 3250 3150
+NoConn ~ 5050 5250
+NoConn ~ 5050 5350
+NoConn ~ 5050 5450
+NoConn ~ 5050 5550
+NoConn ~ 3250 3550
+NoConn ~ 3250 3650
 $EndSCHEMATC

Commit message: Please be right
Connections:
- net 3V3: now also C19.1, D3.1 (K); no longer D3.2 (A)
- net GND: now also D3.2 (A); no longer D3.1 (K)
Other:
- note added: "Battery Babysitter Connector"
- note removed: "Battery Babysitter \nConnector"
- moved on the sheet: C1, C10, C11, C12, C19, C2, C3, C4, C5, C6, C7, C8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

Commit message: I think this is going well
Parts:
- C1, C14, C2, C3, C4: footprint Capacitor_SMD:C_1206_3216Metric_Pad1.42x1.75mm_HandSolder -> Capacitor_SMD:C_1206_3216Metric_Pad1.33x1.80mm_HandSolder
- C10, C11, C13, C15, C18, C5, C6, C7, C8, C9: footprint Capacitor_SMD:C_0805_2012Metric_Pad1.15x1.40mm_HandSolder -> Capacitor_SMD:C_0805_2012Metric_Pad1.18x1.45mm_HandSolder
- C17: footprint Capacitor_SMD:C_1210_3225Metric_Pad1.42x2.65mm_HandSolder -> Capacitor_SMD:C_1210_3225Metric_Pad1.33x2.70mm_HandSolder
- R1, R10, R11, R2, R3, R4, R5, R6, R9: footprint Resistor_SMD:R_0805_2012Metric_Pad1.15x1.40mm_HandSolder -> Resistor_SMD:R_0805_2012Metric_Pad1.20x1.40mm_HandSolder
- Re1, Rf1: footprint Resistor_SMD:R_0805_2012Metric_Pad1.15x1.40mm_HandSolder -> Resistor_SMD:R_0815_2038Metric_Pad1.20x4.05mm_HandSolder
Changed lines of the file:
@@
 F 0 "C13" H 9015 3196 50  0000 L CNN
 F 1 "0.1uF" H 9015 3105 50  0000 L CNN
-F 2 "Capacitor_SMD:C_0805_2012Metric_Pad1.15x1.40mm_HandSolder" H 8938 3000 50  0001 C CNN
+F 2 "Capacitor_SMD:C_0805_2012Metric_Pad1.18x1.45mm_HandSolder" H 8938 3000 50  0001 C CNN
 F 3 "~" H 8900 3150 50  0001 C CNN
 	1    8900 3150
@@
 F 0 "R10" H 1093 1300 50  0000 L BNN
 F 1 "62" H 1184 1300 50  0000 C TNN
-F 2 "Resistor_SMD:R_0805_2012Metric_Pad1.15x1.40mm_HandSolder" V 1230 1300 50  0001 C CNN
+F 2 "Resistor_SMD:R_0805_2012Metric_Pad1.20x1.40mm_HandSolder" V 1230 1300 50  0001 C CNN
 F 3 "~" H 1300 1300 50  0001 C CNN
 	1    1300 1300
@@
 F 0 "C18" H 10915 5896 50  0000 L CNN
 F 1 "0.1uF" H 10915 5805 50  0000 L CNN
-F 2 "Capacitor_SMD:C_0805_2012Metric_Pad1.15x1.40mm_HandSolder" H 10838 5700 50  0001 C CNN
+F 2 "Capacitor_SMD:C_0805_2012Metric_Pad1.18x1.45mm_HandSolder" H 10838 5700 50  0001 C CNN
 F 3 "~" H 10800 5850 50  0001 C CNN
 	1    10800 5850
@@
 F 0 "Re1" V 9420 4746 50  0000 L CNN
 F 1 "10k" V 9420 4655 50  0000 C CNN
-F 2 "Resistor_SMD:R_0805_2012Metric_Pad1.15x1.40mm_HandSolder" V 9280 4700 50  0001 C CNN
+F 2 "Resistor_SMD:R_0815_2038Metric_Pad1.20x4.05mm_HandSolder" V 9280 4700 50  0001 C CNN
 F 3 "~" H 9350 4700 50  0001 C CNN
 	1    9350 4700
@@
 F 0 "Rf1" V 9143 5100 50  0000 C TNN
 F 1 "10k" V 9234 5100 50  0000 C TNN
-F 2 "Resistor_SMD:R_0805_2012Metric_Pad1.15x1.40mm_HandSolder" V 9280 5100 50  0001 C CNN
+F 2 "Resistor_SMD:R_0815_2038Metric_Pad1.20x4.05mm_HandSolder" V 9280 5100 50  0001 C CNN
 F 3 "~" H 9350 5100 50  0001 C CNN
 	1    9350 5100
@@
 F 0 "R1" H 968 5396 50  0000 L CNN
 F 1 "62" H 968 5305 50  0000 L CNN
-F 2 "Resistor_SMD:R_0805_2012Metric_Pad1.15x1.40mm_HandSolder" V 940 5340 50  0001 C CNN
+F 2 "Resistor_SMD:R_0805_2012Metric_Pad1.20x1.40mm_HandSolder" V 940 5340 50  0001 C CNN
 F 3 "~" H 900 5350 50  0001 C CNN
 	1    900  5350
@@
 F 0 "R2" H 968 5746 50  0000 L CNN
 F 1 "62" H 968 5655 50  0000 L CNN
-F 2 "Resistor_SMD:R_0805_2012Metric_Pad1.15x1.40mm_HandSolder" V 940 5690 50  0001 C CNN
+F 2 "Resistor_SMD:R_0805_2012Metric_Pad1.20x1.40mm_HandSolder" V 940 5690 50  0001 C CNN
 F 3 "~" H 900 5700 50  0001 C CNN
 	1    900  5700
@@
 F 0 "C3" H 1015 4146 50  0000 L CNN
 F 1 "1uF" H 1015 4055 50  0000 L CNN
-F 2 "Capacitor_SMD:C_1206_3216Metric_Pad1.42x1.75mm_HandSolder" H 938 3950 50  0001 C CNN
+F 2 "Capacitor_SMD:C_1206_3216Metric_Pad1.33x1.80mm_HandSolder" H 938 3950 50  0001 C CNN
 F 3 "~" H 900 4100 50  0001 C CNN
 	1    900  4100
@@
 F 0 "R5" H 968 3796 50  0000 L CNN
 F 1 "10k" H 968 3705 50  0000 L CNN
-F 2 "Resistor_SMD:R_0805_2012Metric_Pad1.15x1.40mm_HandSolder" V 940 3740 50  0001 C CNN
+F 2 "Resistor_SMD:R_0805_2012Metric_Pad1.20x1.40mm_HandSolder" V 940 3740 50  0001 C CNN
 F 3 "~" H 900 3750 50  0001 C CNN
 	1    900  3750
@@
 F 0 "C1" H 915 1396 50  0000 L CNN
 F 1 "1uF" H 915 1305 50  0000 L CNN
-F 2 "Capacitor_SMD:C_1206_3216Metric_Pad1.42x1.75mm_HandSolder" H 838 1200 50  0001 C CNN
+F 2 "Capacitor_SMD:C_1206_3216Metric_Pad1.33x1.80mm_HandSolder" H 838 1200 50  0001 C CNN
 F 3 "~" H 800 1350 50  0001 C CNN
 	1    800  1350
@@
 F 0 "R3" H 868 1046 50  0000 L CNN
 F 1 "10k" H 868 955 50  0000 L CNN
-F 2 "Resistor_SMD:R_0805_2012Metric_Pad1.15x1.40mm_HandSolder" V 840 990 50  0001 C CNN
+F 2 "Resistor_SMD:R_0805_2012Metric_Pad1.20x1.40mm_HandSolder" V 840 990 50  0001 C CNN
 F 3 "~" H 800 1000 50  0001 C CNN
 	1    800  1000
@@
 F 0 "C2" H 965 2746 50  0000 L CNN
 F 1 "1uF" H 965 2655 50  0000 L CNN
-F 2 "Capacitor_SMD:C_1206_3216Metric_Pad1.42x1.75mm_HandSolder" H 888 2550 50  0001 C CNN
+F 2 "Capacitor_SMD:C_1206_3216Metric_Pad1.33x1.80mm_HandSolder" H 888 2550 50  0001 C CNN
 F 3 "~" H 850 2700 50  0001 C CNN
 	1    850  2700
@@
 F 0 "R4" H 918 2396 50  0000 L CNN
 F 1 "10k" H 918 2305 50  0000 L CNN
-F 2 "Resistor_SMD:R_0805_2012Metric_Pad1.15x1.40mm_HandSolder" V 890 2340 50  0001 C CNN
+F 2 "Resistor_SMD:R_0805_2012Metric_Pad1.20x1.40mm_HandSolder" V 890 2340 50  0001 C CNN
 F 3 "~" H 850 2350 50  0001 C CNN
 	1    850  2350
@@
 F 0 "C15" H 9352 6000 50  0000 R TNN
 F 1 "0.1uF" H 9261 6000 50  0000 C BNN
-F 2 "Capacitor_SMD:C_0805_2012Metric_Pad1.15x1.40mm_HandSolder" H 9138 5850 50  0001 C CNN
+F 2 "Capacitor_SMD:C_0805_2012Metric_Pad1.18x1.45mm_HandSolder" H 9138 5850 50  0001 C CNN
 F 3 "~" H 9100 6000 50  0001 C CNN
 	1    9100 6000
@@
 F 0 "C17" H 9715 6046 50  0000 L CNN
 F 1 "0.0068uF" H 9715 5955 50  0000 L CNN
-F 2 "Capacitor_SMD:C_1210_3225Metric_Pad1.42x2.65mm_HandSolder" H 9638 5850 50  0001 C CNN
+F 2 "Capacitor_SMD:C_1210_3225Metric_Pad1.33x2.70mm_HandSolder" H 9638 5850 50  0001 C CNN
 F 3 "~" H 9600 6000 50  0001 C CNN
 	1    9600 6000
@@
 F 0 "C14" H 9465 1946 50  0000 L CNN
 F 1 "10uF" H 9465 1855 50  0000 L CNN
-F 2 "Capacitor_SMD:C_1206_3216Metric_Pad1.42x1.75mm_HandSolder" H 9388 1750 50  0001 C CNN
+F 2 "Capacitor_SMD:C_1206_3216Metric_Pad1.33x1.80mm_HandSolder" H 9388 1750 50  0001 C CNN
 F 3 "~" H 9350 1900 50  0001 C CNN
 	1    9350 1900
@@
 F 0 "C8" H 6515 1746 50  0000 L CNN
 F 1 "0.1uF" H 6515 1655 50  0000 L CNN
-F 2 "Capacitor_SMD:C_0805_2012Metric_Pad1.15x1.40mm_HandSolder" H 6438 1550 50  0001 C CNN
+F 2 "Capacitor_SMD:C_0805_2012Metric_Pad1.18x1.45mm_HandSolder" H 6438 1550 50  0001 C CNN
 F 3 "~" H 6400 1700 50  0001 C CNN
 	1    6400 1700
@@
 F 0 "C9" H 6765 1746 50  0000 L CNN
 F 1 "0.1uF" H 6765 1655 50  0000 L CNN
-F 2 "Capacitor_SMD:C_0805_2012Metric_Pad1.15x1.40mm_HandSolder" H 6688 1550 50  0001 C CNN
+F 2 "Capacitor_SMD:C_0805_2012Metric_Pad1.18x1.45mm_HandSolder" H 6688 1550 50  0001 C CNN
 F 3 "~" H 6650 1700 50  0001 C CNN
 	1    6650 1700
@@
 F 0 "C10" H 7015 1746 50  0000 L CNN
 F 1 "0.1uF" H 7015 1655 50  0000 L CNN
-F 2 "Capacitor_SMD:C_0805_2012Metric_Pad1.15x1.40mm_HandSolder" H 6938 1550 50  0001 C CNN
+F 2 "Capacitor_SMD:C_0805_2012Metric_Pad1.18x1.45mm_HandSolder" H 6938 1550 50  0001 C CNN
 F 3 "~" H 6900 1700 50  0001 C CNN
 	1    6900 1700
@@
 F 0 "C11" H 7265 1746 50  0000 L CNN
 F 1 "0.1uF" H 7265 1655 50  0000 L CNN
-F 2 "Capacitor_SMD:C_0805_2012Metric_Pad1.15x1.40mm_HandSolder" H 7188 1550 50  0001 C CNN
+F 2 "Capacitor_SMD:C_0805_2012Metric_Pad1.18x1.45mm_HandSolder" H 7188 1550 50  0001 C CNN
 F 3 "~" H 7150 1700 50  0001 C CNN
 	1    7150 1700
@@
 F 0 "C6" H 6015 1746 50  0000 L CNN
 F 1 "0.1uF" H 6015 1655 50  0000 L CNN
-F 2 "Capacitor_SMD:C_0805_2012Metric_Pad1.15x1.40mm_HandSolder" H 5938 1550 50  0001 C CNN
+F 2 "Capacitor_SMD:C_0805_2012Metric_Pad1.18x1.45mm_HandSolder" H 5938 1550 50  0001 C CNN
 F 3 "~" H 5900 1700 50  0001 C CNN
 	1    5900 1700
@@
 F 0 "C7" H 6265 1746 50  0000 L CNN
 F 1 "0.1uF" H 6265 1655 50  0000 L CNN
-F 2 "Capacitor_SMD:C_0805_2012Metric_Pad1.15x1.40mm_HandSolder" H 6188 1550 50  0001 C CNN
+F 2 "Capacitor_SMD:C_0805_2012Metric_Pad1.18x1.45mm_HandSolder" H 6188 1550 50  0001 C CNN
 F 3 "~" H 6150 1700 50  0001 C CNN
 	1    6150 1700
@@
 F 0 "C5" H 3115 2396 50  0000 L CNN
 F 1 "0.1uF" H 3115 2305 50  0000 L CNN
-F 2 "Capacitor_SMD:C_0805_2012Metric_Pad1.15x1.40mm_HandSolder" H 3038 2200 50  0001 C CNN
+F 2 "Capacitor_SMD:C_0805_2012Metric_Pad1.18x1.45mm_HandSolder" H 3038 2200 50  0001 C CNN
 F 3 "~" H 3000 2350 50  0001 C CNN
 	1    3000 2350
@@
 F 0 "C4" H 2865 2396 50  0000 L CNN
 F 1 "1uF" H 2865 2305 50  0000 L CNN
-F 2 "Capacitor_SMD:C_1206_3216Metric_Pad1.42x1.75mm_HandSolder" H 2788 2200 50  0001 C CNN
+F 2 "Capacitor_SMD:C_1206_3216Metric_Pad1.33x1.80mm_HandSolder" H 2788 2200 50  0001 C CNN
 F 3 "~" H 2750 2350 50  0001 C CNN
 	1    2750 2350
@@
 F 0 "R6" H 2518 2146 50  0000 L CNN
 F 1 "510" H 2518 2055 50  0000 L CNN
-F 2 "Resistor_SMD:R_0805_2012Metric_Pad1.15x1.40mm_HandSolder" V 2490 2090 50  0001 C CNN
+F 2 "Resistor_SMD:R_0805_2012Metric_Pad1.20x1.40mm_HandSolder" V 2490 2090 50  0001 C CNN
 F 3 "~" H 2450 2100 50  0001 C CNN
 	1    2450 2100
@@
 F 0 "R9" H 1143 2650 50  0000 L BNN
 F 1 "62" H 1234 2650 50  0000 C TNN
-F 2 "Resistor_SMD:R_0805_2012Metric_Pad1.15x1.40mm_HandSolder" V 1280 2650 50  0001 C CNN
+F 2 "Resistor_SMD:R_0805_2012Metric_Pad1.20x1.40mm_HandSolder" V 1280 2650 50  0001 C CNN
 F 3 "~" H 1350 2650 50  0001 C CNN
 	1    1350 2650
@@
 F 0 "R11" H 1243 4100 50  0000 L BNN
 F 1 "62" H 1334 4100 50  0000 C TNN
-F 2 "Resistor_SMD:R_0805_2012Metric_Pad1.15x1.40mm_HandSolder" V 1380 4100 50  0001 C CNN
+F 2 "Resistor_SMD:R_0805_2012Metric_Pad1.20x1.40mm_HandSolder" V 1380 4100 50  0001 C CNN
 F 3 "~" H 1450 4100 50  0001 C CNN
 	1    1450 4100

Commit message: Cha Cha Cha Changes
Parts:
- J1: footprint Connector_PinHeader_1.00mm:PinHeader_1x06_P1.00mm_Vertical -> Connector_PinHeader_2.54mm:PinHeader_1x06_P2.54mm_Vertical
- J2, J3: footprint Connector_PinHeader_1.00mm:PinHeader_1x02_P1.00mm_Vertical -> Connector_PinHeader_2.54mm:PinHeader_1x02_P2.54mm_Vertical
- J5: footprint Connector_PinHeader_1.00mm:PinHeader_1x04_P1.00mm_Vertical -> Connector_PinHeader_2.54mm:PinHeader_1x04_P2.54mm_Vertical
Changed lines of the file:
@@
 F 0 "J1" H 6856 4028 50  0000 C CNN
 F 1 "Battery Babysitter" V 6856 3937 50  0000 R CNN
-F 2 "Connector_PinHeader_1.00mm:PinHeader_1x06_P1.00mm_Vertical" H 6750 3750 50  0001 C CNN
+F 2 "Connector_PinHeader_2.54mm:PinHeader_1x06_P2.54mm_Vertical" H 6750 3750 50  0001 C CNN
 F 3 "~" H 6750 3750 50  0001 C CNN
 	1    6750 3750
@@
 F 0 "J3" H 2980 1292 50  0000 L CNN
 F 1 "BOOT0" H 2980 1201 50  0000 L CNN
-F 2 "Connector_PinHeader_1.00mm:PinHeader_1x02_P1.00mm_Vertical" H 2900 1300 50  0001 C CNN
+F 2 "Connector_PinHeader_2.54mm:PinHeader_1x02_P2.54mm_Vertical" H 2900 1300 50  0001 C CNN
 F 3 "~" H 2900 1300 50  0001 C CNN
 	1    2900 1300
@@
 	1    0    0    -1
 $EndComp
-$Comp
-L Connector_Generic:Conn_01x04 J5
-U 1 1 5FBD623E
-P 1050 7100
-F 0 "J5" H 968 6675 50  0000 C CNN
-F 1 "Programmer" H 968 6766 50  0000 C CNN
-F 2 "Connector_PinHeader_1.00mm:PinHeader_1x04_P1.00mm_Vertical" H 1050 7100 50  0001 C CNN
-F 3 "~" H 1050 7100 50  0001 C CNN
-	1    1050 7100
-	-1   0    0    1
-$EndComp
-Text GLabel 1250 7000 2    50   Input ~ 0
-SWDIO
 Text GLabel 1250 6900 2    50   Input ~ 0
 SWCLK
-Text GLabel 1250 7100 2    50   Input ~ 0
-3V3
-$Comp
-L power:GND #PWR0103
-U 1 1 5FBFA3D2
-P 1250 7200
-F 0 "#PWR0103" H 1250 6950 50  0001 C CNN
-F 1 "GND" H 1255 7027 50  0000 C CNN
-F 2 "" H 1250 7200 50  0001 C CNN
-F 3 "" H 1250 7200 50  0001 C CNN
-	1    1250 7200
-	1    0    0    -1
-$EndComp
 Text Notes 7150 6900 0    118  ~ 0
 Snow-weAR Goggles\n
@@
 F 0 "J2" H 7930 3842 50  0000 L CNN
 F 1 "BB_SYSOFF" V 7930 3751 50  0000 R CNN
-F 2 "Connector_PinHeader_1.00mm:PinHeader_1x02_P1.00mm_Vertical" H 7850 3850 50  0001 C CNN
+F 2 "Connector_PinHeader_2.54mm:PinHeader_1x02_P2.54mm_Vertical" H 7850 3850 50  0001 C CNN
 F 3 "~" H 7850 3850 50  0001 C CNN
 	1    7850 3850
@@
 Wire Notes Line
 	7200 4300 7200 5150
+$Comp
+L power:GND #PWR0103
+U 1 1 5FBFA3D2
+P 1250 7200
+F 0 "#PWR0103" H 1250 6950 50  0001 C CNN
+F 1 "GND" H 1255 7027 50  0000 C CNN
+F 2 "" H 1250 7200 50  0001 C CNN
+F 3 "" H 1250 7200 50  0001 C CNN
+	1    1250 7200
+	1    0    0    -1
+$EndComp
+Text GLabel 1250 7100 2    50   Input ~ 0
+3V3
+Text GLabel 1250 7000 2    50   Input ~ 0
+SWDIO
+$Comp
+L Connector_Generic:Conn_01x04 J5
+U 1 1 5FBD623E
+P 1050 7100
+F 0 "J5" H 968 6675 50  0000 C CNN
+F 1 "Programmer" H 968 6766 50  0000 C CNN
+F 2 "Connector_PinHeader_2.54mm:PinHeader_1x04_P2.54mm_Vertical" H 1050 7100 50  0001 C CNN
+F 3 "~" H 1050 7100 50  0001 C CNN
+	1    1050 7100
+	-1   0    0    1
+$EndComp
 $EndSCHEMATC
